Commit message: Update sensor_support.xacro

File: iqr_4m_description/urdf/sensor_support.xacro (robot description, xacro)
@@ -28,5 +28,5 @@
     <link name="os_sensor"/>
     <joint name="lidar_joint" type="fixed">
-      <origin xyz="0.0 0.0 0.47322" rpy="0 0 0"/>
+      <origin xyz="0.0 0.0 0.43722" rpy="0 0 0"/>
       <parent link="${prefix}_link"/>
       <child link="os_sensor"/>
